File: tmc2660/tmc2660-quadrigotion.sch (KiCad schematic (older format))
At the start: 15 parts, among them P3 Motor, U1 TMC2660

Commit message: Use smaller connector. JST XH is sufficient for the currents at hand, no need for JST VH
o Also: size adaption. The smaller connector allows to make the board a little
  narrower.
o Add copper pour for VMOT.
Parts:
- P3: footprint Connectors_JST:JST_VH_B4P-VH_4x3.96mm_Vertical -> Connectors_JST:JST_XH_B04B-XH-A_04x2.50mm_Straight
Changed lines of the file:
@@
 LIBS:tmc2660
 LIBS:Connector
+LIBS:tmc2660-quadrigotion-cache
 EELAYER 26 0
 EELAYER END
@@
 F 0 "P3" H 5500 3550 50  0000 C CNN
 F 1 "Motor" V 5600 3300 50  0000 C CNN
-F 2 "Connectors_JST:JST_VH_B4P-VH_4x3.96mm_Vertical" H 5500 3300 60  0001 C CNN
+F 2 "Connectors_JST:JST_XH_B04B-XH-A_04x2.50mm_Straight" H 5500 3300 60  0001 C CNN
 F 3 "" H 5500 3300 60  0000 C CNN
 	1    5500 3300
