File: tmc2660/tmc2660-mono.kicad_pcb (KiCad board)
At the start: 4 copper layers, 25 x 40 mm, 19 parts, among them J100 0R, P100 Motor, U100 TMC2660

Commit message: More preparation for cloning.
Parts:
- M100, M101: renamed from REF**; value M2.5 -> Mount
- moved C104 0.51 mm to (139.2, 49.7)
Routing:
- net /TMC2660-Block/~EN: track 33.4 -> 30.8 mm
- net /TMC2660-Block/CS: track 31.7 -> 29.1 mm
- net /TMC2660-Block/SCLK: track 29.9 -> 27.5 mm
- net /TMC2660-Block/GLOBAL_MISO: track 28.3 -> 26.0 mm
- net /TMC2660-Block/MOSI: track 19.3 -> 17.8 mm
- net /TMC2660-Block/MISO: track 18.7 -> 17.6 mm
Changed lines of the file:
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@@
-(kicad_pcb (version 20170922) (host pcbnew "(2017-11-14 revision d504a8bdd)-master")
+(kicad_pcb (version 20170922) (host pcbnew "(2017-11-16 revision 9d2389fc7)-fix-save-board")
   (general
     (thickness 1.6)
@@
     (39 F.Mask user)
     (40 Dwgs.User user)
-    (41 Cmts.User user)
+    (41 Cmts.User user hide)
     (42 Eco1.User user)
     (43 Eco2.User user)
@@
     (user_trace_width 1.2)
     (trace_clearance 0.127)
-    (zone_clearance 0.254)
+    (zone_clearance 0.4)
     (zone_45_only no)
     (trace_min 0.2)
@@
     (tags "mounting hole 2.7mm no annular m2.5")
     (attr virtual)
-    (fp_text reference REF** (at 0 -3.7) (layer F.SilkS)
-      (effects (font (size 1 1) (thickness 0.15)))
-    )
-    (fp_text value M2.5 (at 4.064 -4.318) (layer F.Fab)
+    (fp_text reference M100 (at 0 -3.7) (layer F.SilkS)
+      (effects (font (size 1 1) (thickness 0.15)))
+    )
+    (fp_text value Mount (at 4.064 -4.318) (layer F.Fab)
       (effects (font (size 1 1) (thickness 0.15)))
     )
@@
     (tags "mounting hole 2.7mm no annular m2.5")
     (attr virtual)
-    (fp_text reference REF** (at 0.254 5.106) (layer F.SilkS)
-      (effects (font (size 1 1) (thickness 0.15)))
-    )
-    (fp_text value M2.5 (at 0 3.7) (layer F.Fab)
+    (fp_text reference M101 (at 0.254 5.106) (layer F.SilkS)
+      (effects (font (size 1 1) (thickness 0.15)))
+    )
+    (fp_text value Mount (at 0 3.7) (layer F.Fab)
       (effects (font (size 1 1) (thickness 0.15)))
     )
@@
   )
   (module Capacitors_SMD:C_0805 (layer F.Cu)
-    (at 139.192 49.2125)
+    (at 139.192 49.7205)
     (descr "Capacitor SMD 0805, reflow soldering, AVX (see smccp.pdf)")
     (tags "capacitor 0805")
@@
   (gr_line (start 142 31.623) (end 142 71.628) (layer Edge.Cuts) (width 0.1))
   (gr_line (start 117 31.623) (end 142 31.623) (layer Edge.Cuts) (width 0.1))
+  (via (at 117.4115 51.943) (size 0.6) (drill 0.4) (layers F.Cu B.Cu) (net 1))
   (via (at 133.477 61.722) (size 0.6) (drill 0.4) (layers F.Cu B.Cu) (net 1))
   (via (at 138.176 66.421) (size 0.6) (drill 0.4) (layers F.Cu B.Cu) (net 1))
@@
   (segment (start 129.8575 48.506) (end 129.8575 47.1685) (width 0.6) (layer F.Cu) (net 1))
   (segment (start 129.8575 47.1685) (end 130.544 46.482) (width 0.6) (layer F.Cu) (net 1))
-  (via (at 117.602 48.387) (size 0.6) (drill 0.4) (layers F.Cu B.Cu) (net 1))
   (via (at 121.285 45.339) (size 0.6) (drill 0.4) (layers F.Cu B.Cu) (net 1))
   (via (at 122.047 44.45) (size 0.6) (drill 0.4) (layers F.Cu B.Cu) (net 1))
@@
   (segment (start 128.778 63.246) (end 131.191 63.246) (width 0.4) (layer In1.Cu) (net 7))
   (segment (start 128.778 63.246) (end 128.766 63.246) (width 0.4) (layer F.Cu) (net 7))
-  (segment (start 131.953 64.008) (end 143.129 64.008) (width 0.4) (layer In1.Cu) (net 7))
+  (segment (start 131.953 64.008) (end 142 64.008) (width 0.4) (layer In1.Cu) (net 7))
   (segment (start 128.2575 61.621462) (end 130.175 63.538962) (width 0.4) (layer F.Cu) (net 8))
   (segment (start 128.2575 60.206) (end 128.2575 61.621462) (width 0.4) (layer F.Cu) (net 8))
   (segment (start 130.175 63.538962) (end 130.175 64.008) (width 0.4) (layer F.Cu) (net 8))
-  (segment (start 128.27 64.008) (end 115.443 64.008) (width 0.4) (layer In1.Cu) (net 8))
+  (segment (start 128.27 64.008) (end 117 64.008) (width 0.4) (layer In1.Cu) (net 8))
   (via (at 130.175 64.008) (size 0.6) (drill 0.4) (layers F.Cu B.Cu) (net 8))
   (segment (start 130.175 64.008) (end 128.27 64.008) (width 0.4) (layer In1.Cu) (net 8))
@@
   (segment (start 129.0575 61.4935) (end 129.54 61.976) (width 0.4) (layer F.Cu) (net 9))
   (segment (start 127 61.976) (end 126.365 62.611) (width 0.4) (layer In1.Cu) (net 9))
-  (segment (start 126.365 62.611) (end 115.697 62.611) (width 0.4) (layer In1.Cu) (net 9))
+  (segment (start 126.365 62.611) (end 117 62.611) (width 0.4) (layer In1.Cu) (net 9))
   (via (at 129.54 61.976) (size 0.6) (drill 0.4) (layers F.Cu B.Cu) (net 9))
   (segment (start 132.588 61.976) (end 133.223 62.611) (width 0.4) (layer In1.Cu) (net 9))
   (segment (start 129.54 61.976) (end 127 61.976) (width 0.4) (layer In1.Cu) (net 9))
   (segment (start 129.54 61.976) (end 132.588 61.976) (width 0.4) (layer In1.Cu) (net 9))
-  (segment (start 133.223 62.611) (end 143.129 62.611) (width 0.4) (layer In1.Cu) (net 9))
+  (segment (start 133.223 62.611) (end 142 62.611) (width 0.4) (layer In1.Cu) (net 9))
   (segment (start 131.826 62.611) (end 132.08 62.865) (width 0.4) (layer In1.Cu) (net 10))
   (via (at 132.08 62.865) (size 0.6) (drill 0.4) (layers F.Cu B.Cu) (net 10))
@@
   (segment (start 130.6575 60.206) (end 130.6575 61.074602) (width 0.4) (layer F.Cu) (net 10))
   (segment (start 130.6575 61.074602) (end 130.915899 61.333001) (width 0.4) (layer F.Cu) (net 10))
-  (segment (start 127.381 63.246) (end 115.57 63.246) (width 0.4) (layer In1.Cu) (net 10))
+  (segment (start 127.381 63.246) (end 117 63.246) (width 0.4) (layer In1.Cu) (net 10))
   (segment (start 128.016 62.611) (end 127.381 63.246) (width 0.4) (layer In1.Cu) (net 10))
   (segment (start 130.683 62.611) (end 128.016 62.611) (width 0.4) (layer In1.Cu) (net 10))
-  (segment (start 132.461 63.246) (end 143.129 63.246) (width 0.4) (layer In1.Cu) (net 10))
+  (segment (start 132.461 63.246) (end 142 63.246) (width 0.4) (layer In1.Cu) (net 10))
   (segment (start 131.826 62.611) (end 132.461 63.246) (width 0.4) (layer In1.Cu) (net 10))
   (segment (start 131.107264 62.611) (end 131.826 62.611) (width 0.4) (layer In1.Cu) (net 10))
@@
   (segment (start 132.969 62.826038) (end 132.969 64.980736) (width 0.4) (layer F.Cu) (net 11))
   (segment (start 132.969 64.980736) (end 132.969 65.405) (width 0.4) (layer F.Cu) (net 11))
-  (segment (start 132.969 65.405) (end 143.256 65.405) (width 0.4) (layer In1.Cu) (net 11))
-  (segment (start 132.969 65.405) (end 115.697 65.405) (width 0.4) (layer In1.Cu) (net 11))
+  (segment (start 132.969 65.405) (end 142 65.405) (width 0.4) (layer In1.Cu) (net 11))
+  (segment (start 132.969 65.405) (end 117 65.405) (width 0.4) (layer In1.Cu) (net 11))
   (via (at 132.969 65.405) (size 0.6) (drill 0.4) (layers F.Cu B.Cu) (net 11))
   (segment (start 128.397 64.377) (end 129.02 64.377) (width 0.4) (layer F.Cu) (net 6))
   (segment (start 129.02 64.377) (end 129.286 64.643) (width 0.4) (layer F.Cu) (net 6))
   (via (at 129.286 64.643) (size 0.6) (drill 0.4) (layers F.Cu B.Cu) (net 6))
-  (segment (start 129.54 64.643) (end 142.875 64.643) (width 0.4) (layer In1.Cu) (net 6))
-  (segment (start 129.54 64.643) (end 115.57 64.643) (width 0.4) (layer In1.Cu) (net 6))
+  (segment (start 129.54 64.643) (end 142 64.643) (width 0.4) (layer In1.Cu) (net 6))
+  (segment (start 129.54 64.643) (end 117 64.643) (width 0.4) (layer In1.Cu) (net 6))
   (zone (net 15) (net_name /TMC2660-Block/A2) (layer B.Cu) (hatch edge 0.508)
     (priority 1)
@@
     (polygon
       (pts
-        (xy 118.11 53.34) (xy 123.698 53.34) (xy 123.698 60.96) (xy 118.11 60.96)
+        (xy 118.11 51.562) (xy 123.698 51.562) (xy 123.698 60.96) (xy 118.11 60.96)
       )
     )
@@
       (pts
         (xy 130.556 59.563) (xy 130.556 49.657) (xy 135.636 49.657) (xy 135.636 60.96) (xy 133.985 60.96)
-      )
-    )
-  )
-  (zone (net 16) (net_name /TMC2660-Block/B2) (layer In1.Cu) (hatch edge 0.508)
-    (priority 1)
-    (connect_pads yes (clearance 0.4))
-    (min_thickness 0.254)
-    (fill yes (arc_segments 16) (thermal_gap 0.508) (thermal_bridge_width 0.508))
-    (polygon
-      (pts
-        (xy 136.144 53.34) (xy 141.224 53.34) (xy 141.224 60.96) (xy 136.144 60.96)
       )
     )
@@
     (polygon
       (pts
-        (xy 116.332 49.022) (xy 118.999 49.022) (xy 123.063 44.069) (xy 116.332 44.069)
+        (xy 116.3955 47.8155) (xy 119.0625 47.8155) (xy 123.063 44.069) (xy 116.332 44.069)
       )
     )
@@
     (polygon
       (pts
-        (xy 143.129 60.96) (xy 143.002 71.755) (xy 115.824 71.755) (xy 115.697 60.96) (xy 129.286 49.657)
-        (xy 130.302 49.657)
+        (xy 137.922 51.4985) (xy 143.0655 51.4985) (xy 143.002 71.755) (xy 115.824 71.755) (xy 115.8875 51.4985)
+        (xy 120.7135 51.4985) (xy 129.286 49.657) (xy 130.302 49.657)
       )
     )
@@
     (polygon
       (pts
-        (xy 116.332 44.069) (xy 123.063 44.069) (xy 118.999 49.022) (xy 116.332 49.022)
+        (xy 116.332 44.069) (xy 123.063 44.069) (xy 118.999 47.879) (xy 116.332 47.879)
       )
     )
@@
       )
     )
+  )
+  (zone (net 0) (net_name "") (layer Cmts.User) (hatch edge 0.508)
+    (connect_pads (clearance 0.254))
+    (min_thickness 0.254)
+    (fill yes (arc_segments 16) (thermal_gap 0.508) (thermal_bridge_width 0.508))
+    (polygon
+      (pts
+        (xy 145.415 73.533) (xy 145.415 30.353) (xy 114.1095 30.353) (xy 109.347 30.353) (xy 109.347 73.025)
+      )
+    )
+  )
+  (zone (net 16) (net_name /TMC2660-Block/B2) (layer In1.Cu) (hatch edge 0.508)
+    (priority 1)
+    (connect_pads yes (clearance 0.4))
+    (min_thickness 0.254)
+    (fill yes (arc_segments 16) (thermal_gap 0.508) (thermal_bridge_width 0.508))
+    (polygon
+      (pts
+        (xy 136.144 51.562) (xy 141.6685 51.562) (xy 141.6685 60.96) (xy 136.144 60.96)
+      )
+    )
