File: tmc2660/tmc2660-quad.sch (KiCad schematic (older format))
At the start: 5 parts, among them J1 Power, J2 DataIn, M0 Mount, M1 Mount

Commit message: Integrate grounded mounting hole.
Parts:
- M1: footprint Mounting_Holes:MountingHole_2.7mm_M2.5 -> Mounting_Holes:MountingHole_2.7mm_M2.5_Pad; symbol Mechanical:Mounting_Hole -> Mechanical:Mounting_Hole_PAD
Changed lines of the file:
@@
 EESchema Schematic File Version 4
-LIBS:tmc2660-quad-cache
 EELAYER 26 0
 EELAYER END
@@
 L Mechanical:Mounting_Hole M0
 U 1 1 5A1112B3
-P 2300 4600
-F 0 "M0" H 2358 4720 50  0000 L CNN
-F 1 "Mount" H 2358 4629 50  0000 L CNN
-F 2 "Mounting_Holes:MountingHole_2.7mm_M2.5" H 2500 4600 50  0001 C CNN
-F 3 "~" H 2500 4600 50  0001 C CNN
-	1    2300 4600
-	1    0    0    -1
-$EndComp
-$Comp
-L Mechanical:Mounting_Hole M1
+P 2300 4550
+F 0 "M0" H 2250 4700 50  0000 L CNN
+F 1 "Mount" H 2200 4800 50  0000 L CNN
+F 2 "Mounting_Holes:MountingHole_2.7mm_M2.5" H 2500 4550 50  0001 C CNN
+F 3 "~" H 2500 4550 50  0001 C CNN
+	1    2300 4550
+	1    0    0    -1
+$EndComp
+$Comp
+L Mechanical:Mounting_Hole_PAD M1
 U 1 1 5A1112BA
 P 2700 4600
-F 0 "M1" H 2758 4720 50  0000 L CNN
-F 1 "Mount" H 2758 4629 50  0000 L CNN
-F 2 "Mounting_Holes:MountingHole_2.7mm_M2.5" H 2900 4600 50  0001 C CNN
+F 0 "M1" H 2700 4800 50  0000 L CNN
+F 1 "Mount" H 2600 4900 50  0000 L CNN
+F 2 "Mounting_Holes:MountingHole_2.7mm_M2.5_Pad" H 2900 4600 50  0001 C CNN
 F 3 "~" H 2900 4600 50  0001 C CNN
 	1    2700 4600
@@
 Text Label 2700 1600 0    60   ~ 0
 PowerIn
+$Comp
+L power:GND #PWR?
+U 1 1 5A1C0ADE
+P 2700 4700
+F 0 "#PWR?" H 2700 4450 50  0001 C CNN
+F 1 "GND" V 2705 4572 50  0000 R CNN
+F 2 "" H 2700 4700 50  0001 C CNN
+F 3 "" H 2700 4700 50  0001 C CNN
+	1    2700 4700
+	1    0    0    -1
+$EndComp
 $EndSCHEMATC

Commit message: Use surface-mount IDC connector for easier PCB heatsink mount.
Parts:
- J2: footprint Connectors_IDC:IDC-Header_2x08_Pitch2.54mm_Straight -> Quadrigotion:IDC_Header_SMD_16pins
Changed lines of the file:
@@
 EESchema Schematic File Version 4
+LIBS:tmc2660-quad-cache
 EELAYER 26 0
 EELAYER END
@@
 F 0 "J2" H 2550 2825 50  0000 C CNN
 F 1 "DataIn" H 2550 2916 50  0000 C CNN
-F 2 "Connectors_IDC:IDC-Header_2x08_Pitch2.54mm_Straight" H 2500 3450 50  0001 C CNN
+F 2 "Quadrigotion:IDC_Header_SMD_16pins" H 2500 3450 50  0001 C CNN
 F 3 "~" H 2500 3450 50  0001 C CNN
 	1    2500 3450
@@
 PowerIn
 $Comp
-L power:GND #PWR?
+L power:GND #PWR02
 U 1 1 5A1C0ADE
 P 2700 4700
-F 0 "#PWR?" H 2700 4450 50  0001 C CNN
+F 0 "#PWR02" H 2700 4450 50  0001 C CNN
 F 1 "GND" V 2705 4572 50  0000 R CNN
 F 2 "" H 2700 4700 50  0001 C CNN
