File: tmc2660/tmc2660-block-200.sch (KiCad schematic (older format))
At the start: 18 parts, among them J200 0R, M200 Mount, M201 Mount, P200 Motor, U200 TMC2660

Commit message: Wire up quad according to new MISO/MOSI sequence.
- Also, add basic STEP/DIR and a capacitor.
Parts:
- renumbered C201 to C200, C200 to C201, C203 to C202, C202 to C203, C206 to C205, C207 to C206, C205 to C207, R201 to R200, R200 to R201, R203 to R202, R202 to R203
Connections:
- net labels added: START_MOSI
- net labels removed: GLOBAL_MISO
- wire segments 51 -> 50
Other:
- note added: "Jumper on\nhighest popuplated"
- note removed: "Optional"
- moved on the sheet: J200
Changed lines of the file:
@@
 EESchema Schematic File Version 4
-LIBS:tmc2660-mono-cache
+LIBS:tmc2660-quad-cache
 EELAYER 26 0
 EELAYER END
 $Descr A4 11693 8268
 encoding utf-8
-Sheet 2 2
+Sheet 2 5
 Title ""
 Date ""
@@
 $EndDescr
 $Comp
-L device:C C202
+L device:C C203
 U 1 1 5A0CA5B9
 P 4250 2250
-F 0 "C202" H 4275 2350 50  0000 L CNN
+F 0 "C203" H 4275 2350 50  0000 L CNN
 F 1 "10u" H 4275 2150 50  0000 L CNN
 F 2 "Capacitors_SMD:C_1206" H 4288 2100 30  0001 C CNN
@@
 $EndComp
 $Comp
-L device:C C203
+L device:C C202
 U 1 1 5A0CA5C0
 P 4250 3100
-F 0 "C203" H 4275 3200 50  0000 L CNN
+F 0 "C202" H 4275 3200 50  0000 L CNN
 F 1 "10u" H 4275 3000 50  0000 L CNN
 F 2 "Capacitors_SMD:C_1206" H 4288 2950 30  0001 C CNN
@@
 $EndComp
 $Comp
-L device:C C206
+L device:C C205
 U 1 1 5A0CA5D3
 P 2900 1800
-F 0 "C206" H 2650 1900 50  0000 L CNN
+F 0 "C205" H 2650 1900 50  0000 L CNN
 F 1 "100n" H 2700 1700 50  0000 L CNN
 F 2 "Capacitors_SMD:C_0805" H 2938 1650 30  0001 C CNN
@@
 Connection ~ 3400 3150
 $Comp
-L device:R R202
+L device:R R203
 U 1 1 5A0CA5F8
 P 3550 2700
-F 0 "R202" V 3650 2700 50  0000 C CNN
+F 0 "R203" V 3650 2700 50  0000 C CNN
 F 1 "10R" V 3550 2700 50  0000 C CNN
 F 2 "Resistors_SMD:R_0603" V 3480 2700 30  0001 C CNN
@@
 $EndComp
 $Comp
-L device:R R203
+L device:R R202
 U 1 1 5A0CA5FF
 P 3550 3550
-F 0 "R203" V 3450 3550 50  0000 C CNN
+F 0 "R202" V 3450 3550 50  0000 C CNN
 F 1 "10R" V 3550 3550 50  0000 C CNN
 F 2 "Resistors_SMD:R_0603" V 3480 3550 30  0001 C CNN
@@
 $EndComp
 $Comp
-L device:C C207
+L device:C C206
 U 1 1 5A0CA648
 P 2250 3700
-F 0 "C207" H 1950 3700 50  0000 L CNN
+F 0 "C206" H 1950 3700 50  0000 L CNN
 F 1 "100n" H 2050 3600 50  0000 L CNN
 F 2 "Capacitors_SMD:C_0603" H 2288 3550 30  0001 C CNN
@@
 $EndComp
 Wire Wire Line
-	1500 2150 2350 2150
+	2050 2150 2350 2150
 Wire Wire Line
 	2350 3500 2300 3500
@@
 	2300 3500 2300 3550
 Wire Wire Line
-	2300 3550 2000 3550
+	2000 3550 2300 3550
 $Comp
 L power:GND #PWR0109
@@
 $EndComp
 $Comp
-L device:R R201
+L device:R R200
 U 1 1 5A0CA66C
 P 3950 3700
-F 0 "R201" V 3850 3650 50  0000 C CNN
+F 0 "R200" V 3850 3650 50  0000 C CNN
 F 1 "0.075" V 3950 3700 50  0000 C CNN
 F 2 "Resistors_SMD:R_2512" V 3880 3700 30  0001 C CNN
@@
 $EndComp
 $Comp
-L device:R R200
+L device:R R201
 U 1 1 5A0CA673
 P 3950 2850
-F 0 "R200" V 3850 2850 50  0000 C CNN
+F 0 "R201" V 3850 2850 50  0000 C CNN
 F 1 "0.075" V 3950 2850 50  0000 C CNN
 F 2 "Resistors_SMD:R_2512" V 3880 2850 30  0001 C CNN
@@
 	2250 2250 2350 2250
 $Comp
-L device:C_Small C200
+L device:C_Small C201
 U 1 1 5A0CA67B
 P 3950 2700
-F 0 "C200" V 3800 2600 50  0000 L CNN
+F 0 "C201" V 3800 2600 50  0000 L CNN
 F 1 "10n" V 3900 2750 50  0000 L CNN
 F 2 "Capacitors_SMD:C_0603" H 3988 2550 30  0001 C CNN
@@
 	3400 2450 3600 2450
 $Comp
-L device:C_Small C201
+L device:C_Small C200
 U 1 1 5A0CA683
 P 3950 3550
-F 0 "C201" V 4000 3600 50  0000 L CNN
+F 0 "C200" V 4000 3600 50  0000 L CNN
 F 1 "10n" V 4000 3350 50  0000 L CNN
 F 2 "Capacitors_SMD:C_0603" H 3988 3400 30  0001 C CNN
@@
 DIR
 Wire Wire Line
-	1250 2400 2350 2400
+	1850 2400 2350 2400
 Wire Wire Line
 	2350 2500 1250 2500
@@
 Connection ~ 3800 2700
 $Comp
-L device:CP C205
+L device:CP C207
 U 1 1 5A0CA6BD
 P 3500 1700
-F 0 "C205" H 3525 1800 50  0000 L CNN
+F 0 "C207" H 3525 1800 50  0000 L CNN
 F 1 "100u" H 3400 1900 50  0000 L CNN
 F 2 "Capacitors_THT:CP_Radial_D10.0mm_P5.00mm" H 3538 1550 30  0001 C CNN
@@
 	3200 1850 3500 1850
 Connection ~ 3350 1850
-Text Notes 1600 2350 0    60   ~ 0
-Optional
+Text Notes 600  2400 0    51   ~ 0
+Jumper on\nhighest popuplated
 Text HLabel 3750 1550 2    60   Input ~ 0
 VMot
@@
 Text HLabel 2000 3550 0    60   Input ~ 0
 VCC
-Text HLabel 1500 2150 0    60   Input ~ 0
+Text HLabel 2050 2150 0    60   Input ~ 0
 ~EN
 $Comp
 L device:R J200
 U 1 1 5A0CA6C8
-P 1400 2300
-F 0 "J200" V 1450 2100 50  0000 C CNN
-F 1 "0R" V 1400 2300 50  0000 C CNN
-F 2 "Resistors_SMD:R_0603" V 1330 2300 30  0001 C CNN
-F 3 "" H 1400 2300 30  0000 C CNN
-	1    1400 2300
-	0    -1   -1   0
-$EndComp
-Text HLabel 1250 2300 0    60   Input ~ 0
-GLOBAL_MISO
-Text HLabel 1250 2400 0    60   Input ~ 0
+P 1450 2350
+F 0 "J200" H 1550 2500 50  0000 C CNN
+F 1 "0R" V 1450 2350 50  0000 C CNN
+F 2 "Resistors_SMD:R_0603" V 1380 2350 30  0001 C CNN
+F 3 "" H 1450 2350 30  0000 C CNN
+	1    1450 2350
+	1    0    0    -1
+$EndComp
+Text HLabel 1250 2200 0    60   Input ~ 0
+START_MOSI
+Text HLabel 1850 2400 0    60   Input ~ 0
 MISO
-Wire Wire Line
-	1550 2300 1600 2300
-Wire Wire Line
-	1600 2300 1600 2400
-Connection ~ 1600 2400
 Text HLabel 1250 2500 0    60   Input ~ 0
 MOSI
@@
 	1    0    0    -1
 $EndComp
+Wire Wire Line
+	1250 2200 1450 2200
+Connection ~ 1450 2500
 $EndSCHEMATC

Commit message: Update tmc2660-quad with new template.
o Start out with a tmc2660-quad-baseline that is filled
  in with zones and tracks from the template.
o The separation from baseline and template allows faster
  updates later.
Parts:
- C202, C203: Voltage (none) -> 50V
- C204: footprint Capacitors_SMD:C_0805 -> Capacitors_SMD:C_0603; Voltage (none) -> 50V
- C205: footprint Capacitors_SMD:C_0805 -> Capacitors_SMD:C_0603; Voltage (none) -> 16V
- C206, C208: Voltage (none) -> 16V
- C207: value 100u -> 180u; footprint Capacitors_THT:CP_Radial_D10.0mm_P5.00mm -> Capacitors_THT:CP_Radial_D8.0mm_P3.50mm; DigiKey (none) -> 565-3911-ND; Voltage (none) -> 35V
Connections:
- net labels added: VHS
- wire segments 50 -> 44
Other:
- moved on the sheet: C200, C201, C202, C203, C205, P200, R200, R201, R202, R203

Commit message: Integrate grounded mounting hole.
Parts:
- C202, C203: DigiKey (none) -> 1276-6736-1-ND
- C204: footprint Capacitors_SMD:C_0603 -> Capacitors_SMD:C_0805; DigiKey (none) -> 1276-2450-2-ND
- C205, C206: footprint Capacitors_SMD:C_0603 -> Capacitors_SMD:C_0805; DigiKey (none) -> 1276-2450-2-ND; Voltage 16V -> >= 16V
- M201: footprint Mounting_Holes:MountingHole_2.7mm_M2.5 -> Mounting_Holes:MountingHole_2.7mm_M2.5_Pad; symbol Mechanical:Mounting_Hole -> Mechanical:Mounting_Hole_PAD
- R200, R201: Alternative 100mOhm (none) -> CRM2512-JX-R100ELFCT-ND; DigiKey (none) -> CSRN2512FK75L0CT-ND
Other:
- note added: "Sense Resistors alternatively\nalso with 100mOhm"
Changed lines of the file:
@@
 EESchema Schematic File Version 4
-LIBS:tmc2660-mono-cache
 EELAYER 26 0
 EELAYER END
@@
 F 3 "" H 4400 2300 60  0000 C CNN
 F 4 "50V" H 4400 2300 60  0001 C CNN "Voltage"
+F 5 "1276-6736-1-ND" H 4400 2300 60  0001 C CNN "DigiKey"
 	1    4400 2300
 	1    0    0    -1
@@
 F 3 "" H 4100 2300 60  0000 C CNN
 F 4 "50V" H 4100 2300 60  0001 C CNN "Voltage"
+F 5 "1276-6736-1-ND" H 4100 2300 60  0001 C CNN "DigiKey"
 	1    4100 2300
 	1    0    0    -1
@@
 F 0 "C205" H 2800 2000 50  0000 L CNN
 F 1 "100n" H 2700 1800 50  0000 L CNN
-F 2 "Capacitors_SMD:C_0603" H 2938 1550 30  0001 C CNN
+F 2 "Capacitors_SMD:C_0805" H 2938 1550 30  0001 C CNN
 F 3 "" H 2900 1700 60  0000 C CNN
-F 4 "16V" H 2900 1700 60  0001 C CNN "Voltage"
+F 4 ">= 16V" H 2900 1700 60  0001 C CNN "Voltage"
+F 5 "1276-2450-2-ND" H 2900 1700 60  0001 C CNN "DigiKey"
 	1    2900 1700
 	1    0    0    -1
@@
 F 0 "C204" H 3150 2000 50  0000 L CNN
 F 1 "100n" H 3150 1900 50  0000 L CNN
-F 2 "Capacitors_SMD:C_0603" H 3238 1550 30  0001 C CNN
+F 2 "Capacitors_SMD:C_0805" H 3238 1550 30  0001 C CNN
 F 3 "" H 3200 1700 60  0000 C CNN
 F 4 "50V" H 3200 1700 60  0001 C CNN "Voltage"
+F 5 "1276-2450-2-ND" H 3200 1700 60  0001 C CNN "DigiKey"
 	1    3200 1700
 	1    0    0    -1
@@
 F 0 "C206" H 1950 3700 50  0000 L CNN
 F 1 "100n" H 2050 3600 50  0000 L CNN
-F 2 "Capacitors_SMD:C_0603" H 2288 3550 30  0001 C CNN
+F 2 "Capacitors_SMD:C_0805" H 2288 3550 30  0001 C CNN
 F 3 "" H 2250 3700 60  0000 C CNN
-F 4 "16V" H 2250 3700 60  0001 C CNN "Voltage"
+F 4 ">= 16V" H 2250 3700 60  0001 C CNN "Voltage"
+F 5 "1276-2450-2-ND" H 2250 3700 60  0001 C CNN "DigiKey"
 	1    2250 3700
 	1    0    0    -1
@@
 F 2 "Resistors_SMD:R_2512" V 4330 3500 30  0001 C CNN
 F 3 "" H 4400 3500 30  0000 C CNN
+F 4 "CSRN2512FK75L0CT-ND" H 4400 3500 60  0001 C CNN "DigiKey"
+F 5 "CRM2512-JX-R100ELFCT-ND" H 4400 3500 60  0001 C CNN "Alternative 100mOhm"
 	1    4400 3500
 	-1   0    0    1
@@
 F 2 "Resistors_SMD:R_2512" V 4330 2950 30  0001 C CNN
 F 3 "" H 4400 2950 30  0000 C CNN
+F 4 "CSRN2512FK75L0CT-ND" H 4400 2950 60  0001 C CNN "DigiKey"
+F 5 "CRM2512-JX-R100ELFCT-ND" H 4400 2950 60  0001 C CNN "Alternative 100mOhm"
 	1    4400 2950
 	1    0    0    -1
@@
 L Mechanical:Mounting_Hole M200
 U 1 1 5A0FBC47
-P 1250 4300
-F 0 "M200" H 1308 4420 50  0000 L CNN
-F 1 "Mount" H 1308 4329 50  0000 L CNN
-F 2 "Mounting_Holes:MountingHole_2.7mm_M2.5" H 1450 4300 50  0001 C CNN
-F 3 "~" H 1450 4300 50  0001 C CNN
-	1    1250 4300
-	1    0    0    -1
-$EndComp
-$Comp
-L Mechanical:Mounting_Hole M201
+P 1250 4250
+F 0 "M200" H 1150 4400 50  0000 L CNN
+F 1 "Mount" H 1308 4279 50  0000 L CNN
+F 2 "Mounting_Holes:MountingHole_2.7mm_M2.5" H 1450 4250 50  0001 C CNN
+F 3 "~" H 1450 4250 50  0001 C CNN
+	1    1250 4250
+	1    0    0    -1
+$EndComp
+$Comp
+L Mechanical:Mounting_Hole_PAD M201
 U 1 1 5A0FBD0F
 P 1650 4300
-F 0 "M201" H 1708 4420 50  0000 L CNN
+F 0 "M201" H 1550 4500 50  0000 L CNN
 F 1 "Mount" H 1708 4329 50  0000 L CNN
-F 2 "Mounting_Holes:MountingHole_2.7mm_M2.5" H 1850 4300 50  0001 C CNN
+F 2 "Mounting_Holes:MountingHole_2.7mm_M2.5_Pad" H 1850 4300 50  0001 C CNN
 F 3 "~" H 1850 4300 50  0001 C CNN
 	1    1650 4300
@@
 Text Label 2900 1950 1    39   ~ 0
 VHS
+Text Notes 4500 3750 0    51   ~ 0
+Sense Resistors alternatively\nalso with 100mOhm
+$Comp
+L power:GND #PWR?
+U 1 1 5A1C342B
+P 1650 4400
+F 0 "#PWR?" H 1650 4150 50  0001 C CNN
+F 1 "GND" H 1650 4250 50  0000 C CNN
+F 2 "" H 1650 4400 60  0000 C CNN
+F 3 "" H 1650 4400 60  0000 C CNN
+	1    1650 4400
+	1    0    0    -1
+$EndComp
 $EndSCHEMATC

Commit message: Move VMOT 100nF input stabilisator for VHS voltage regulator close to pin.
o Re-number the 100nF capacitors that they show up in an increasing numbers
o Use opportunity to move silkscreen of 10uF capacitors out of via's harms way.
Parts:
- renumbered C205 to C204, C204 to C205
Connections:
- wire segments 44 -> 63
Changed lines of the file:
@@
 EESchema Schematic File Version 4
-LIBS:tmc2660-quad-cache
 EELAYER 26 0
 EELAYER END
 $Descr A4 11693 8268
 encoding utf-8
-Sheet 2 5
+Sheet 2 2
 Title ""
 Date ""
@@
 $EndComp
 $Comp
-L power:GND #PWR026
+L power:GND #PWR0101
 U 1 1 5A0CA5C7
 P 3800 3050
-F 0 "#PWR026" H 3800 2800 50  0001 C CNN
+F 0 "#PWR0101" H 3800 2800 50  0001 C CNN
 F 1 "GND" H 3800 2900 50  0000 C CNN
 F 2 "" H 3800 3050 60  0000 C CNN
@@
 $EndComp
 $Comp
-L power:GND #PWR027
+L power:GND #PWR0102
 U 1 1 5A0CA5CD
 P 4400 2450
-F 0 "#PWR027" H 4400 2200 50  0001 C CNN
+F 0 "#PWR0102" H 4400 2200 50  0001 C CNN
 F 1 "GND" H 4400 2300 50  0000 C CNN
 F 2 "" H 4400 2450 60  0000 C CNN
@@
 $EndComp
 $Comp
-L device:C C205
+L device:C C204
 U 1 1 5A0CA5D3
 P 2900 1700
-F 0 "C205" H 2800 2000 50  0000 L CNN
+F 0 "C204" H 2800 2000 50  0000 L CNN
 F 1 "100n" H 2700 1800 50  0000 L CNN
 F 2 "Capacitors_SMD:C_0805" H 2938 1550 30  0001 C CNN
@@
 $EndComp
 $Comp
-L device:C C204
+L device:C C205
 U 1 1 5A0CA5DE
 P 3200 1700
-F 0 "C204" H 3150 2000 50  0000 L CNN
+F 0 "C205" H 3150 2000 50  0000 L CNN
 F 1 "100n" H 3150 1900 50  0000 L CNN
 F 2 "Capacitors_SMD:C_0805" H 3238 1550 30  0001 C CNN
@@
 $EndComp
 $Comp
-L power:GND #PWR028
+L power:GND #PWR0103
 U 1 1 5A0CA5E6
 P 3350 1850
-F 0 "#PWR028" H 3350 1600 50  0001 C CNN
+F 0 "#PWR0103" H 3350 1600 50  0001 C CNN
 F 1 "GND" H 3450 1750 50  0000 C CNN
 F 2 "" H 3350 1850 60  0000 C CNN
@@
 $EndComp
 $Comp
-L power:GND #PWR029
+L power:GND #PWR0104
 U 1 1 5A0CA5EF
 P 2800 3800
-F 0 "#PWR029" H 2800 3550 50  0001 C CNN
+F 0 "#PWR0104" H 2800 3550 50  0001 C CNN
 F 1 "GND" H 2800 3650 50  0000 C CNN
 F 2 "" H 2800 3800 60  0000 C CNN
@@
 $EndComp
 $Comp
-L power:GND #PWR030
+L power:GND #PWR0105
 U 1 1 5A0CA606
 P 3750 3950
-F 0 "#PWR030" H 3750 3700 50  0001 C CNN
+F 0 "#PWR0105" H 3750 3700 50  0001 C CNN
 F 1 "GND" H 3750 3800 50  0000 C CNN
 F 2 "" H 3750 3950 60  0000 C CNN
@@
 $EndComp
 $Comp
-L power:GND #PWR031
+L power:GND #PWR0106
 U 1 1 5A0CA623
 P 2050 3400
-F 0 "#PWR031" H 2050 3150 50  0001 C CNN
+F 0 "#PWR0106" H 2050 3150 50  0001 C CNN
 F 1 "GND" H 2050 3250 50  0000 C CNN
 F 2 "" H 2050 3400 60  0000 C CNN
@@
 $EndComp
 $Comp
-L power:GND #PWR032
+L power:GND #PWR0107
 U 1 1 5A0CA642
 P 2250 3850
-F 0 "#PWR032" H 2250 3600 50  0001 C CNN
+F 0 "#PWR0107" H 2250 3600 50  0001 C CNN
 F 1 "GND" H 2250 3700 50  0000 C CNN
 F 2 "" H 2250 3850 60  0000 C CNN
@@
 NoConn ~ 2350 3250
 $Comp
-L power:GND #PWR033
+L power:GND #PWR0108
 U 1 1 5A0CA65B
 P 2250 2250
-F 0 "#PWR033" H 2250 2000 50  0001 C CNN
+F 0 "#PWR0108" H 2250 2000 50  0001 C CNN
 F 1 "GND" H 2250 2100 50  0000 C CNN
 F 2 "" H 2250 2250 60  0000 C CNN
@@
 $EndComp
 $Comp
-L power:GND #PWR034
+L power:GND #PWR0109
 U 1 1 5A0CA666
 P 2500 3800
-F 0 "#PWR034" H 2500 3550 50  0001 C CNN
+F 0 "#PWR0109" H 2500 3550 50  0001 C CNN
 F 1 "GND" H 2450 3650 50  0000 C CNN
 F 2 "" H 2500 3800 60  0000 C CNN
@@
 Connection ~ 3050 1550
 Wire Wire Line
-	2700 3800 2900 3800
+	2700 3800 2800 3800
 Connection ~ 2800 3800
 Connection ~ 3400 2250
@@
 	3400 2250 3600 2250
 Wire Wire Line
-	3400 3300 3400 3450
+	3400 3300 3400 3350
 Connection ~ 3400 3350
 Wire Wire Line
-	3400 3050 3400 3200
+	3400 3050 3400 3100
 Connection ~ 3400 3100
 Wire Wire Line
-	3400 2450 3400 2600
+	3400 2450 3400 2500
 Connection ~ 3400 2500
 Wire Wire Line
-	3400 2200 3400 2350
+	3400 2200 3400 2250
 Connection ~ 3400 2300
 Wire Wire Line
@@
 	2300 3500 2300 3550
 Wire Wire Line
-	2000 3550 2300 3550
+	2000 3550 2250 3550
 Wire Wire Line
 	2250 2250 2350 2250
 Wire Wire Line
 	3400 2450 3600 2450
-Connection ~ 3400 3300
 Connection ~ 3400 3400
 Wire Wire Line
-	3400 3550 3800 3550
+	3400 3550 3750 3550
 Wire Wire Line
 	3400 2700 3800 2700
 Wire Wire Line
-	3400 2800 4400 2800
-Connection ~ 3400 3050
+	3400 2800 4250 2800
 Wire Wire Line
 	2350 2850 1950 2850
@@
 	1850 2400 2350 2400
 Wire Wire Line
-	1250 2500 2350 2500
+	1250 2500 1450 2500
 Wire Wire Line
 	2350 2600 1250 2600
@@
 Connection ~ 3200 1550
 Wire Wire Line
-	3200 1850 3500 1850
+	3200 1850 3350 1850
 Connection ~ 3350 1850
 Connection ~ 3500 1550
 Wire Wire Line
-	2900 1550 3750 1550
+	2900 1550 3050 1550
 Wire Wire Line
 	3400 3100 3600 3100
@@
 Connection ~ 4250 2800
 $Comp
-L power:GND #PWR035
+L power:GND #PWR01
 U 1 1 5A17CB15
 P 4600 3200
-F 0 "#PWR035" H 4600 2950 50  0001 C CNN
+F 0 "#PWR01" H 4600 2950 50  0001 C CNN
 F 1 "GND" H 4600 3050 50  0000 C CNN
 F 2 "" H 4600 3200 60  0000 C CNN
@@
 Connection ~ 3800 2700
 Wire Wire Line
-	4400 3100 4400 3350
+	4400 3100 4400 3200
 Wire Wire Line
 	4400 3200 4600 3200
 Connection ~ 4400 3200
 Wire Wire Line
-	3400 3650 4400 3650
+	3400 3650 4200 3650
 Wire Wire Line
 	4100 3550 4200 3550
@@
 Wire Wire Line
 	4100 2450 4400 2450
-Connection ~ 4400 2450
 Wire Wire Line
 	2900 1850 2900 1950
@@
 Sense Resistors alternatively\nalso with 100mOhm
 $Comp
-L power:GND #PWR036
+L power:GND #PWR?
 U 1 1 5A1C342B
 P 1650 4400
-F 0 "#PWR036" H 1650 4150 50  0001 C CNN
+F 0 "#PWR?" H 1650 4150 50  0001 C CNN
 F 1 "GND" H 1650 4250 50  0000 C CNN
 F 2 "" H 1650 4400 60  0000 C CNN
@@
 	1    0    0    -1
 $EndComp
+Wire Wire Line
+	3050 1550 3200 1550
+Wire Wire Line
+	2800 3800 2900 3800
+Wire Wire Line
+	3400 2250 3400 2300
+Wire Wire Line
+	3400 2550 3400 2600
+Wire Wire Line
+	3400 3150 3400 3200
+Wire Wire Line
+	3400 3350 3400 3400
+Wire Wire Line
+	3400 3100 3400 3150
+Wire Wire Line
+	3400 2500 3400 2550
+Wire Wire Line
+	3400 2300 3400 2350
+Wire Wire Line
+	2250 3550 2300 3550
+Wire Wire Line
+	3400 3400 3400 3450
+Wire Wire Line
+	3200 1550 3500 1550
+Wire Wire Line
+	3350 1850 3500 1850
+Wire Wire Line
+	3500 1550 3750 1550
+Wire Wire Line
+	1450 2500 2350 2500
+Wire Wire Line
+	4250 2800 4400 2800
+Wire Wire Line
+	4400 3200 4400 3350
+Wire Wire Line
+	4200 3650 4400 3650
+Wire Wire Line
+	3750 3550 3800 3550
 $EndSCHEMATC
